File: CCA/v1r0/scale_cca/scale_cca.kicad_sch (KiCad schematic)
At the start: 22 parts

Commit message: as built v1r0
Other:
- note added: "0.1W / SK6805 1.1W (5v/0.22a) / CCA"
- note added: "VCC: 3.5-5.5V"
- note removed: "3.5-5.5V"
Changed lines of the file:
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@@
   (title_block
     (title "Scale CCA")
-    (date "2021-08-14")
+    (date "2021-08-15")
     (rev "v1r0")
   )
@@
     (stroke (width 0) (type solid) (color 0 0 0 0))
   )
-  (text "3.5-5.5V" (at 86.36 35.56 180)
-    (effects (font (size 1.27 1.27)) (justify right bottom))
+  (text "VCC: 3.5-5.5V" (at 17.78 21.59 0)
+    (effects (font (size 1.27 1.27)) (justify left bottom))
+  )
+  (text "0.1W / SK6805\n1.1W (5v/0.22a) / CCA" (at 17.78 30.48 0)
+    (effects (font (size 1.27 1.27)) (justify left bottom))
   )
   (label "DIN" (at 64.77 69.85 180)
