File: CCA/v1r1/scale_cca/scale_cca.kicad_pcb (KiCad board)
At the start: 2 copper layers, 22.2 x 35.8 mm, 22 parts

Commit message: v1r1 as fabricated
Parts:
- removed C2: C_Small, Capacitor_SMD:C_0805_2012Metric
- added D12: SK6805, SK6805_2020:LED_SK6805_2.0x2.0mm, F.Cu at (43.0, 50.7)
- added D13: SK6805, SK6805_2020:LED_SK6805_2.0x2.0mm, F.Cu at (44.6, 46.1)
- C1: value C_Small -> 100 nF
- moved D7 14.3 mm to (28.4, 46.1)
- moved D6 13.0 mm to (40.2, 43.6)
- moved D11 12.9 mm to (40.2, 54.7)
- moved D9 11.9 mm to (32.8, 54.7)
- moved D10 11.9 mm to (36.5, 57.8)
- moved D8 10.7 mm to (30.0, 50.7)
- moved C1 9.90 mm to (36.5, 43.3), turned to 0 degrees
- moved TP1 8.38 mm to (42.2, 45.6), turned to 80 degrees
- moved TP2 8.38 mm to (30.8, 45.6), turned to 100 degrees
- moved D4 7.67 mm to (36.5, 52.5)
- moved D2 5.79 mm to (32.8, 43.6)
- moved FID2 5.41 mm to (26.5, 41.3)
- moved FID3 5.41 mm to (46.5, 41.3)
- moved TP4 4.08 mm to (28.3, 41.3), turned to 90 degrees
- moved TP3 4.08 mm to (44.8, 41.3), turned to -90 degrees
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Connections:
- D10 pad 4: /DIN -> LED_ROW
- D11 pad 2: unconnected-(D11-Pad2) -> Net-(D11-Pad2)
- D2 pad 2: unconnected-(D2-Pad2) -> Net-(D2-Pad2)
- D3 pad 2: unconnected-(D3-Pad2) -> Net-(D4-Pad4)
- D3 pad 4: /DIN -> Net-(D2-Pad2)
- D4 pad 2: unconnected-(D4-Pad2) -> Net-(D4-Pad2)
- D4 pad 4: Net-(D8-Pad4) -> Net-(D4-Pad4)
- D5 pad 2: Net-(D8-Pad4) -> Net-(D5-Pad2)
- D5 pad 4: /DIN -> Net-(D4-Pad2)
- D6 pad 2: unconnected-(D6-Pad2) -> Net-(D6-Pad2)
- D6 pad 4: Net-(D8-Pad4) -> Net-(D5-Pad2)
- D7 pad 2: unconnected-(D7-Pad2) -> Net-(D7-Pad2)
- D7 pad 4: Net-(D8-Pad4) -> Net-(D6-Pad2)
- D8 pad 2: unconnected-(D8-Pad2) -> Net-(D8-Pad2)
- D8 pad 4: Net-(D8-Pad4) -> Net-(D7-Pad2)
- D9 pad 2: /DOUT -> LED_ROW
- D9 pad 4: Net-(D8-Pad4) -> Net-(D8-Pad2)
Routing:
- net GND: track 0.00 -> 136.8 mm, vias 0 -> 5
- net VCC: track 0.00 -> 100.8 mm, vias 0 -> 4
- net Net-(D6-Pad2): track 0.00 -> 21.1 mm, vias 0 -> 2
- net Net-(D1-Pad2): track 0.00 -> 16.3 mm, vias 0 -> 2
- net /DIN: track 0.00 -> 15.0 mm, vias 0 -> 2
- net Net-(D2-Pad2): track 0.00 -> 13.0 mm, vias 0 -> 2
- net /DOUT: track 0.00 -> 12.4 mm, vias 0 -> 2
- net Net-(D5-Pad2): track 0.00 -> 9.12 mm, vias 0 -> 2
- net Net-(D7-Pad2): track 0.00 -> 6.40 mm
- net Net-(D8-Pad2): track 0.00 -> 5.87 mm
- net LED_ROW: track 0.00 -> 5.48 mm
- net Net-(D4-Pad4): track 0.00 -> 5.16 mm
- net Net-(D12-Pad2): track 0.00 -> 3.70 mm
- net Net-(D11-Pad2): track 0.00 -> 3.67 mm
- net Net-(D10-Pad2): track 0.00 -> 3.39 mm
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Other:
- outline, holes or cut-outs redrawn
- board text added: "Large LED Scalemaille"
- board text added: "v1r1"
- board text removed: "D"
- board text removed: "IN"
- board text removed: "Large v1r1"
- board text removed: "Scalemaille LED"
