File: CCA/v1r1/scale_cca/scale_cca.kicad_sch (KiCad schematic)
At the start: 22 parts

Commit message: v1r1 as fabricated
Parts:
- removed C2: C_Small, Capacitor_SMD:C_0805_2012Metric, symbol Device:C_Small
- added D12, D13: SK6805, SK6805_2020:LED_SK6805_2.0x2.0mm, symbol SK6805_2020:SK6805
- C1: value C_Small -> 100 nF
Connections:
- net DIN: no longer D10.4 (DIN), D3.4 (DIN), D5.4 (DIN)
- net DOUT: now also D13.2 (DOUT); no longer D9.2 (DOUT)
- net GND: now also D12.3 (GND), D13.3 (GND)
- net VCC: now also D12.1 (VDD), D13.1 (VDD)
- net at D3.2 (DOUT): now also D4.4 (DIN)
- net at D7.2 (DOUT): now also D8.4 (DIN)
- net at D4.2 (DOUT): now also D5.4 (DIN)
- net at D8.2 (DOUT): now also D9.4 (DIN)
- net at D2.2 (DOUT): now also D3.4 (DIN)
- net at D11.2 (DOUT): now also D12.4 (DIN)
- net at D6.2 (DOUT): now also D7.4 (DIN)
- new net: D12.2 (DOUT), D13.4 (DIN)
- new net: D5.2 (DOUT), D6.4 (DIN)
- new net LED_ROW: D10.4 (DIN), D9.2 (DOUT)
- no-connect marks 3 -> 0
Other:
- note added: "TBR: 0.1W / SK6805 1.1W (5v/0.22a) / CCA"
- note removed: "0.1W / SK6805 1.1W (5v/0.22a) / CCA"
- note removed: "First equivalent LED: central 4 pixels OR D5 ONLY (if only bottom half of CCA is populated)"
- note removed: "Second equivalent LED: Outer 7 pixels OR D4, D6, D7, D9, D10 (if only bottom half of CCA is populated)"
- moved on the sheet: C1, D10, D11, D2, D3, D4, D5, D6, D7, D8, D9, FID1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
