File: CCA/v1r2/scale_cca/scale_cca.kicad_sch (KiCad schematic)
At the start: 27 parts

Commit message: mold
Parts:
- added C2: 100 nF, Capacitor_SMD:C_0805_2012Metric, symbol Device:C_Small
Connections:
- net GND: now also C2.2
- net VCC: now also C2.1
Changed lines of the file:
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@@
   (junction (at 223.52 27.94) (diameter 1.016) (color 0 0 0 0))
   (junction (at 231.14 27.94) (diameter 1.016) (color 0 0 0 0))
+  (junction (at 240.03 27.94) (diameter 1.016) (color 0 0 0 0))
   (junction (at 267.97 20.32) (diameter 1.016) (color 0 0 0 0))
   (wire (pts (xy 57.15 69.85) (xy 44.45 69.85))
@@
     (pin "1")
   )
+  (symbol (lib_id "power:GND") (at 240.03 33.02 0) (unit 1)
+    (in_bom yes) (on_board yes)
+    (property "Reference" "#PWR0101" (id 0) (at 240.03 39.37 0)
+      (effects (font (size 1.27 1.27)) hide)
+    )
+    (property "Value" "GND" (id 1) (at 240.03 37.3444 0))
+    (property "Footprint" "" (id 2) (at 240.03 33.02 0)
+      (effects (font (size 1.27 1.27)) hide)
+    )
+    (property "Datasheet" "" (id 3) (at 240.03 33.02 0)
+      (effects (font (size 1.27 1.27)) hide)
+    )
+    (pin "1")
+  )
   (symbol (lib_id "power:GND") (at 275.59 22.86 0) (unit 1)
     (in_bom yes) (on_board yes)
@@
     )
     (property "Datasheet" "~" (id 3) (at 223.52 30.48 0)
+      (effects (font (size 1.27 1.27)) hide)
+    )
+    (pin "1")
+    (pin "2")
+  )
+  (symbol (lib_id "Device:C_Small") (at 240.03 30.48 0) (mirror y) (unit 1)
+    (in_bom yes) (on_board yes)
+    (property "Reference" "C2" (id 0) (at 237.7058 29.7191 0)
+      (effects (font (size 1.27 1.27)) (justify left))
+    )
+    (property "Value" "100 nF" (id 1) (at 237.7058 32.0178 0)
+      (effects (font (size 1.27 1.27)) (justify left))
+    )
+    (property "Footprint" "Capacitor_SMD:C_0805_2012Metric" (id 2) (at 240.03 30.48 0)
+      (effects (font (size 1.27 1.27)) hide)
+    )
+    (property "Datasheet" "~" (id 3) (at 240.03 30.48 0)
       (effects (font (size 1.27 1.27)) hide)
     )
@@
       (reference "#PWR033") (unit 1) (value "GND") (footprint "")
     )
+    (path "/741cd794-28c5-475f-ac10-0466a664d375"
+      (reference "#PWR0101") (unit 1) (value "GND") (footprint "")
+    )
     (path "/2a2169c2-dea9-4e60-bd38-0b78970e6364"
       (reference "C1") (unit 1) (value "10 uF") (footprint "Capacitor_SMD:C_0805_2012Metric")
     )
+    (path "/a70699b6-5fd1-47ee-8d79-8b69b6b1dcfd"
+      (reference "C2") (unit 1) (value "100 nF") (footprint "Capacitor_SMD:C_0805_2012Metric")
+    )
     (path "/4bab9a77-dc64-4823-ae84-762ebfd7af8a"
